Commit message: update

File: nav_mecanum_description/urdf/nav_mecanum.urdf.xacro (robot description, xacro)
@@ -9,13 +9,13 @@
   <xacro:arg name="simulation_controllers" default="" />
   <xacro:include filename="$(find nav_mecanum_description)/urdf/nav_mecanum/nav_mecanum_macro.xacro"/>
-  <xacro:include filename="$(find nav_mecanum_description)/urdf/nav_mecanum/nav_mecanum_macro.ros2_control.xacro"/>
+  <!-- <xacro:include filename="$(find nav_mecanum_description)/urdf/nav_mecanum/nav_mecanum_macro.ros2_control.xacro"/> -->
   <!-- create link fixed to the "world" -->
-  <link name="world" />
+  <!-- <link name="odom" /> -->
   <!-- Load robot's macro with parameters -->
   <!-- set prefix if multiple robots are used -->
-  <xacro:nav_mecanum prefix="$(arg prefix)" parent="world" >
+  <xacro:nav_mecanum prefix="$(arg prefix)" parent="odom">
     <origin xyz="0 0 0" rpy="0 0 0" />          <!-- position robot in the world -->
   </xacro:nav_mecanum>
-  <xacro:nav_mecanum_ros2_control
+  <!-- <xacro:nav_mecanum_ros2_control
     name="nav_mecanum"
     prefix="$(arg prefix)"
@@ -24,4 +24,4 @@
     sim_gazebo_classic="$(arg sim_gazebo_classic)"
     sim_gazebo="$(arg sim_gazebo)"
-    simulation_controllers="$(arg simulation_controllers)" />
+    simulation_controllers="$(arg simulation_controllers)" /> -->
 </robot>

File: nav_mecanum_description/urdf/nav_mecanum/nav_mecanum_macro.xacro (robot description, xacro)
@@ -12,5 +12,5 @@
         <origin xyz="0 0 0" rpy="0 0 0" />
         <geometry>
-          <box size="0.6 1 0.2"/>
+          <box size="0.21 0.2 0.07"/>
 <!--           <mesh filename="package://nav_mecanum_description/meshes/nav_mecanum/visual/base_link.dae" /> -->
         </geometry>
@@ -19,5 +19,23 @@
         <origin xyz="0 0 0" rpy="0 0 0" />
         <geometry>
-          <box size="0.6 1 0.2"/>
+          <box size="0.193 0.223 0.07"/>
+<!--           <mesh filename="package://nav_mecanum_description/meshes/nav_mecanum/collision/base_link.stl" /> -->
+        </geometry>
+      </collision>
+    </link>
+    <!-- laser -->
+    <link name="${prefix}laser">
+      <xacro:default_inertial/>
+      <visual>
+        <origin xyz="0 0 0" rpy="0 0 0" />
+        <geometry>
+          <cylinder length="0.04" radius="0.03"/>
+<!--           <mesh filename="package://nav_mecanum_description/meshes/nav_mecanum/visual/base_link.dae" /> -->
+        </geometry>
+      </visual>
+      <collision>
+        <origin xyz="0 0 0" rpy="0 0 0" />
+        <geometry>
+          <cylinder length="0.04" radius="0.03"/>
 <!--           <mesh filename="package://nav_mecanum_description/meshes/nav_mecanum/collision/base_link.stl" /> -->
         </geometry>
@@ -32,5 +50,5 @@
         <origin xyz="0 0 0" rpy="0 0 0" />
         <geometry>
-          <cylinder length="0.1" radius="0.2" />
+          <cylinder length="0.03" radius="0.0375" />
 <!--           <mesh filename="package://nav_mecanum_description/meshes/nav_mecanum/visual/link1.dae" /> -->
         </geometry>
@@ -39,5 +57,5 @@
         <origin xyz="0 0 0" rpy="0 0 0" />
         <geometry>
-          <cylinder length="0.1" radius="0.2" />
+          <cylinder length="0.03" radius="0.0375" />
 <!--           <mesh filename="package://nav_mecanum_description/meshes/nav_mecanum/collision/link1.stl" /> -->
         </geometry>
@@ -52,5 +70,5 @@
         <origin xyz="0 0 0" rpy="0 0 0" />
         <geometry>
-          <cylinder length="0.1" radius="0.2" />
+          <cylinder length="0.03" radius="0.0375" />
 <!--           <mesh filename="package://nav_mecanum_description/meshes/nav_mecanum/visual/link2.dae" /> -->
         </geometry>
@@ -59,5 +77,5 @@
         <origin xyz="0 0 0" rpy="0 0 0" />
         <geometry>
-          <cylinder length="0.1" radius="0.2" />
+          <cylinder length="0.03" radius="0.0375" />
 <!--           <mesh filename="package://nav_mecanum_description/meshes/nav_mecanum/collision/link2.stl"  /> -->
         </geometry>
@@ -72,5 +90,5 @@
         <origin xyz="0 0 0" rpy="0 0 0" />
         <geometry>
-          <cylinder length="0.1" radius="0.2" />
+          <cylinder length="0.03" radius="0.0375" />
 <!--           <mesh filename="package://nav_mecanum_description/meshes/nav_mecanum/visual/link3.dae" /> -->
         </geometry>
@@ -79,5 +97,5 @@
         <origin xyz="0 0 0" rpy="0 0 0" />
         <geometry>
-          <cylinder length="0.1" radius="0.2" />
+          <cylinder length="0.03" radius="0.0375" />
 <!--           <mesh filename="package://nav_mecanum_description/meshes/nav_mecanum/collision/link3.stl"  /> -->
         </geometry>
@@ -92,5 +110,5 @@
         <origin xyz="0 0 0" rpy="0 0 0" />
         <geometry>
-          <cylinder length="0.1" radius="0.2" />
+          <cylinder length="0.03" radius="0.0375" />
 <!--           <mesh filename="package://nav_mecanum_description/meshes/nav_mecanum/visual/link4.dae" /> -->
         </geometry>
@@ -99,5 +117,5 @@
         <origin xyz="0 0 0" rpy="0 0 0" />
         <geometry>
-          <cylinder length="0.1" radius="0.2" />
+          <cylinder length="0.03" radius="0.0375" />
 <!--           <mesh filename="package://nav_mecanum_description/meshes/nav_mecanum/collision/link4.stl"  /> -->
         </geometry>
@@ -107,12 +125,19 @@
     <!-- JOINTS -->
     <!-- base_joint fixes base_link to the environment -->
-    <joint name="${prefix}base_joint" type="fixed">
+    <!-- <joint name="${prefix}base_joint" type="fixed">
       <xacro:insert_block name="origin" />
       <parent link="${parent}" />
       <child link="${prefix}base_link" />
+    </joint> -->
+    <!-- laser -->
+    <joint name="${prefix}laser_joint" type="fixed">
+      <origin xyz="0.09 0 0.055" rpy="0 0 ${pi}" />
+      <parent link="${prefix}base_link" />
+      <child link="${prefix}laser" />
+      <axis xyz="0 0 1" />
     </joint>
     <!-- joint 1 -->
     <joint name="${prefix}left_front_wheel_joint" type="continuous">
-      <origin xyz="0.5 -0.5 0" rpy="0 ${pi/2} 0" />
+      <origin xyz="0.0965 0.1115 -0.0275" rpy="${pi/2} ${pi/2} 0" />
       <parent link="${prefix}base_link" />
       <child link="${prefix}link1" />
@@ -121,5 +146,5 @@
     <!-- joint 2 -->
     <joint name="${prefix}left_rear_wheel_joint" type="continuous">
-      <origin xyz="-0.5 -0.5 0" rpy="0 ${pi/2} 0" />
+      <origin xyz="-0.0965 0.1115 -0.0275" rpy="${pi/2} ${pi/2} 0" />
       <parent link="${prefix}base_link" />
       <child link="${prefix}link2" />
@@ -128,5 +153,5 @@
     <!-- joint 3 -->
     <joint name="${prefix}right_front_wheel_joint" type="continuous">
-      <origin xyz="0.5 0.5 0" rpy="0 ${pi/2} 0" />
+      <origin xyz="0.0965 -0.1115 -0.0275" rpy="${pi/2} ${pi/2} 0" />
       <parent link="${prefix}base_link" />
       <child link="${prefix}link3" />
@@ -135,5 +160,5 @@
     <!-- joint 4 -->
     <joint name="${prefix}right_rear_wheel_joint" type="continuous">
-      <origin xyz="-0.5 0.5 0" rpy="0 ${pi/2} 0" />
+      <origin xyz="-0.0965 -0.1115 -0.0275" rpy="${pi/2} ${pi/2} 0" />
       <parent link="${prefix}base_link" />
       <child link="${prefix}link4" />
